File: Projet_Réveil_électronique.kicad_sch (KiCad schematic)
At the start: 26 parts, among them Q1 AO3400A, U1 XIAO-ESP32-S3-DIP, U2 RV-3028-C7, U3 IS31FL3730, U5 DC56-11EWA, U6 DC56-11EWA

Commit message: [M05] - Finalize KiCad Schematic and PCB
Parts:
- renumbered R4 to R3, R3 to R4
Connections:
- net +3.3V: now also U1.12 (3V3), U2.7 (VDD)
- net GND: now also Button_ALARM2.1, Button_MINUS3.2, U1.13 (GND), U2.5 (VSS); no longer Button_ALARM2.2, Button_MINUS3.1
- net at U6.13 (DIG2_CC): now also U3.23 (C2); no longer U3.21 (C4)
- net at U6.14 (DIG1_CC): now also U3.24 (C1); no longer U3.22 (C3)
- net at U1.4 (PA11_A3_D3): now also Button_SET1.2; no longer Button_ALARM2.1
- net at U5.13 (DIG2_CC): now also U3.21 (C4); no longer U3.23 (C2)
- net at U5.14 (DIG1_CC): now also U3.22 (C3); no longer U3.24 (C1)
- net at U1.8 (PB09_A7_D7_RX): now also Button_MINUS3.1; no longer Button_MINUS3.2
- net at U1.3 (PA10_A2_D2): now also Button_ALARM2.2; no longer Button_SET1.2
Other:
- moved on the sheet: Button_ALARM2, Button_MINUS3, Button_PLUS4, Button_SET1
